Commit message: drone in the canel inside the rice field

File: assembly_1/urdf/assembly_1.urdf.xacro (robot description, xacro)
@@ -1,3 +1,2 @@
-<!--URDF generated by ONSHAPE BY PTC INC, 1.219-->
 <robot name="assembly_1" xmlns:xacro="http://www.ros.org/wiki/xacro">
     <link name="root">
@@ -16,4 +15,11 @@
             </material>
         </visual>
+        <collision>
+            <origin xyz="0.00908956 0.0132281 -0.0575308" rpy="0 -0 0" />
+            <geometry>
+                <mesh filename="package://assembly_1/meshes/Default.stl" scale="1 1 1" />
+            </geometry>
+        </collision>
     </link>
+    <xacro:include filename="$(find assembly_1)/urdf/gps.xacro"/>
 </robot>

Commit message: add gps sensor /navsat

File: assembly_1/urdf/assembly_1.urdf.xacro (robot description, xacro)
@@ -1,2 +1,3 @@
+<?xml version="1.0"?>
 <robot name="assembly_1" xmlns:xacro="http://www.ros.org/wiki/xacro">
     <link name="root">

File: assembly_1/urdf/gps.xacro (robot description, xacro)
@@ -1,14 +1,40 @@
-<robot>
-    <sensor name="my_gps" type="gps">
-  <!-- ensure the sensor is active (required) -->
-  <always_on>true</always_on>
-  <update_rate>30</update_rate>
-  <plugin name="my_gps_plugin" filename="libgazebo_ros_gps_sensor.so">
-    <ros>
-      <!-- publish to /gps/data -->
-      <namespace>/gps</namespace>
-      <remapping>~/out:=data</remapping>
-    </ros>
-  </plugin>
-</sensor>
+<?xml version="1.0"?>
+<robot name="gps_robot" xmlns:xacro="http://www.ros.org/wiki/xacro">
+  <joint name="gps_joint" type="fixed">
+    <!-- the root of the drone or the component that the gps link attched to -->
+    <parent link="root"/>
+     <!-- the gps link  -->
+    <child link="gps"/>
+    <origin xyz="0.3 0.3 0.3" rpy="0 0 0"/>
+  </joint>
+  <link name ="gps">
+    <visual>
+      <geometry>
+        <!-- the box around the drone -->
+        <box size="0.03 0.03 0.01"/>
+      </geometry>
+    </visual>
+    <inertial>
+        <mass value="0.01"/>
+        <!--//rpy rotation ;row, ptich , yaw  -->
+        <origin xyz="0 0 0" rpy="0 0 0"/>
+        <inertia
+            ixx="0.00001"
+            ixy="0"
+            ixz="0"
+            iyy="0.00001"
+            iyz="0"
+            izz="0.00001"/>
+    </inertial>
+  </link>
+  <gazebo reference="gps">
+  <sensor name="navsat_sensor" type="navsat">
+    <always_on>1</always_on>
+    <update_rate>10</update_rate>
+    <topic>navsat</topic>
+  </sensor>
+  </gazebo>
+  <gazebo>
+  <plugin filename="ignition-gazebo-navsat-system" name="ignition::gazebo::systems::NavSat"/>
+  </gazebo>
 </robot>

Commit message: quatcopter motors

File: assembly_1/urdf/assembly_1.urdf.xacro (robot description, xacro)
@@ -16,4 +16,13 @@
             </material>
         </visual>
+        <visual>
+            <origin xyz="0 0 0.02" rpy="0 0 0" />
+            <geometry>
+                <box size="0.18 0.18 0.08"/>
+            </geometry>
+            <material name="body_material">
+                <color rgba="0.2 0.2 0.2 1"/>
+            </material>
+        </visual>
         <collision>
             <origin xyz="0.00908956 0.0132281 -0.0575308" rpy="0 -0 0" />
@@ -23,6 +32,15 @@
         </collision>
     </link>
+    <xacro:include filename="$(find assembly_1)/urdf/actuator.xacro"/>
+    <xacro:quad_arm name="arm_fr" angle="0.785" x="0" y="0"/>
+    <xacro:quad_arm name="arm_fl" angle="2.356" x="0" y="0"/>
+    <xacro:quad_arm name="arm_bl" angle="-2.356" x="0" y="0"/>
+    <xacro:quad_arm name="arm_br" angle="-0.785" x="0" y="0"/>
     <xacro:include filename="$(find assembly_1)/urdf/gps.xacro"/>
     <xacro:include filename="$(find assembly_1)/urdf/imu.xacro"/>
     <xacro:include filename="$(find assembly_1)/urdf/camera.xacro"/>
+    <xacro:include filename="motor1.xacro" />
+    <xacro:include filename="motor2.xacro" />
+    <xacro:include filename="motor3.xacro" />
+    <xacro:include filename="motor4.xacro" />
 </robot>

File: assembly_1/urdf/gps.xacro (robot description, xacro)
@@ -12,5 +12,5 @@
       <geometry>
         <!-- the box around the drone -->
-        <box size="0.03 0.03 0.01"/>
+        <box size="0.3 0.3 0.08"/>
       </geometry>
     </visual>
@@ -35,6 +35,8 @@
   </sensor>
   </gazebo>
-<gazebo>
-  <plugin filename="gz-sim-imu-system" name="gz::sim::systems::Imu"/>
-</gazebo>
+ <plugin
+      filename="gz-sim-navsat-system"
+      name="gz::sim::systems::NavSat">
+  </plugin>
+  <mesh filename="package://assembly_1/meshes/Default.stl"/>
 </robot>

File: assembly_1/urdf/imu.xacro (robot description, xacro)
@@ -32,6 +32,5 @@
     </sensor>
   </gazebo>
-<gazebo>
-    <plugin filename="gz-sim-imu-system" name="gz::sim::systems::Imu"/>
-</gazebo>
+<plugin name="gz::sim::systems::Imu"
+        filename="gz-sim-imu-system"/>
 </robot>
