Commit message: reconnect to px4 with rice_field world

File: assembly_1/install/assembly_1/share/assembly_1/urdf/actuator.xacro (robot description, xacro)
@@ -2,5 +2,5 @@
 <robot xmlns:xacro="http://www.ros.org/wiki/xacro">
   <xacro:macro name="quad_arm" params="name angle x y">
-    <link name="${name}">
+    <link name="actuator_link">
       <inertial>
         <mass value="0.01"/>
@@ -20,5 +20,5 @@
       </collision>
     </link>
-    <joint name="${name}_joint" type="fixed">
+    <joint name="actuator_joint" type="fixed">
       <parent link="base_link"/>
       <child link="${name}"/>
